File: projects/lcduino/lcduino.sch (EAGLE design)
At the start: 19 parts, among them IC1 MEGA32-A, IC2 7805DT, J1 1X2-3.5MM, SW1 SPST_TACT-EVQQ2, T1 2N3904, X1 16MHz

Commit message: some board edits
Parts:
- removed C4: 10uF, rcl:CPOL-US085CS-1AR
- removed C5, C6, C7: .1uF, rcl:C-USC0805K
- removed R1, R4: 1k, adafruit:R-US_R0805
- removed R2: 10k, adafruit:R-US_R0805
- removed R3: 2.2k, adafruit:R-US_R0805
- removed T1: 2N3904, transistor:2N3904
- added JP1, JP2: (no value), adafruit:PINHD-1X8CLEANBIG
- IC1: value MEGA32-A -> MEGA8-AI; device atmel:MEGA32-A -> atmel:MEGA8-AI; MF (none) -> Atmel; MPN (none) -> ATMEGA328P-AU; OC_FARNELL (none) -> 1715486; OC_NEWARK (none) -> 68T2935
- U$1: value (none) -> 10k
Connections:
- removed net N$1: C1.+, IC1.XTAL2, X1.P$2
- removed net N$2: C2.+, IC1.XTAL1, X1.P$1
- new net 0: IC1.PD0(RXD)
- new net 1: IC1.PD1(TXD)
- new net 10: IC1.PB2(SS/OC1B), JP2.4
- new net 11: IC1.PB3(MOSI/OC2), JP2.5
- new net 12: IC1.PB4(MISO), JP2.6
- new net 13: IC1.PB5(SCK)
- new net 2: IC1.PD2(INT0)
- new net 3: IC1.PD3(INT1)
- new net 4: IC1.PD4(XCK/T0)
- new net 5: IC1.PD5(T1)
- new net 6: IC1.PD6(AIN0)
- new net 7: IC1.PD7(AIN1), JP1.4
- new net 8: IC1.PB0(ICP), JP1.6
- new net 9: IC1.PB1(OC1A), JP2.3
- new net A0: IC1.PC0(ADC0)
- new net A1: IC1.PC1(ADC1)
- new net A2: IC1.PC2(ADC2)
- new net A3: IC1.PC3(ADC3)
- new net A4: IC1.PC4(ADC4/SDA)
- new net A5: IC1.PC5(ADC5/SCL)
- new net L3: JP1.3, U$1.S
- new net N$10: IC1.ADC7
- new net N$9: IC1.ADC6
- new net XTAL1: C1.+, IC1.PB6(XTAL1/TOSC1), X1.P$2
- new net XTAL2: C2.+, IC1.PB7(XTAL2/TOSC2), X1.P$1
- net 5V: now also IC1.AVCC, IC1.VCC@1, IC1.VCC@2, JP1.2, JP2.7, U$1.A
- net GND: now also IC1.GND, IC1.GND@1, IC1.GND@2, JP1.1, JP1.5, JP2.8, U$1.E
- net RESET: now also IC1.PC6(/RESET); no longer IC1.RESET
Other:
- moved on the sheet: C1, C2, X1
