File: projects/lcduino/lcduino.brd (EAGLE design)
At the start: 152.4 x 25.4 mm, 19 parts, among them IC1 MEGA32-A, IC2 7805DT, J1 1X2-3.5MM, SW1 SPST_TACT-EVQQ2, T1 2N3904, X1 16MHz

Commit message: some board edits
Parts:
- removed C4: 10uF, rcl:085CS_1AR
- removed C5, C6, C7: .1uF, rcl:C0805K
- removed R1, R4: 1k, adafruit:R0805
- removed R2: 10k, adafruit:R0805
- removed R3: 2.2k, adafruit:R0805
- removed T1: 2N3904, transistor:TO92
- added JP1, JP2: (no value), adafruit:1X08-CLEANBIG
- IC1: value MEGA32-A -> MEGA8-AI; device atmel:TQFP44 -> atmel:TQFP32-08
- U$1: value (none) -> 10k
- moved U$1 55.8 mm to (12.0, 6.82), turned to 180 degrees
- moved D1 24.3 mm to (8.00, 34.0)
- moved IC2 23.1 mm to (15.3, 28.6)
- moved J1 23.0 mm to (4.00, 27.0)
- moved C2 22.8 mm to (34.0, 8.00), turned to 180 degrees
- moved C3 18.7 mm to (16.9, 20.2), turned to 0 degrees
- moved C1 12.2 mm to (19.4, 10.9), turned to 90 degrees
- moved SW1 11.9 mm to (36.1, 28.4), turned to 270 degrees
- moved X1 6.71 mm to (25.0, 11.0)
- moved IC1 6.20 mm to (36.0, 18.0)
Connections:
- net AVCC renamed A4
- net N$1 renamed XTAL1
- net N$2 renamed XTAL2
- net VCC1 renamed 13
- removed net GND1: IC1.18
- removed net GND2: IC1.39
- removed net VCC: IC1.5
- removed net VCC2: IC1.38
- new net 0: IC1.30
- new net 1: IC1.31
- new net 10: IC1.14, JP2.4
- new net 11: IC1.15, JP2.5
- new net 12: IC1.16, JP2.6
- new net 2: IC1.32
- new net 3: IC1.1
- new net 4: IC1.2
- new net 5: IC1.9
- new net 6: IC1.10
- new net 7: IC1.11, JP1.4
- new net 8: IC1.12, JP1.6
- new net 9: IC1.13, JP2.3
- new net A0: IC1.23
- new net A1: IC1.24
- new net A2: IC1.25
- new net A3: IC1.26
- new net A5: IC1.28
- new net L3: JP1.3, U$1.2
- new net N$10: IC1.22
- new net N$9: IC1.19
- net 5V: now also IC1.18, IC1.4, IC1.6, JP1.2, JP2.7, U$1.1
- net GND: now also IC1.21, IC1.3, IC1.5, JP1.1, JP1.5, JP2.8, U$1.3; no longer IC1.28, IC1.6
- net RESET: now also IC1.29; no longer IC1.4
Routing:
- net 5V: track 17.7 -> 136.9 mm
- net 7: track 0.00 -> 28.5 mm
- net 8: track 0.00 -> 24.8 mm
- net 10: track 0.00 -> 20.2 mm
- net 11: track 0.00 -> 19.1 mm
- net 12: track 0.00 -> 18.3 mm
- net XTAL1: track 31.7 -> 13.8 mm
- net 9: track 0.00 -> 13.1 mm
- net XTAL2: track 27.5 -> 18.2 mm
- net L3: track 0.00 -> 3.01 mm
- net VIN: track 4.96 -> 3.28 mm
- net PWRIN: track 5.23 -> 6.02 mm
- added copper zone on layer 1, net GND
Other:
- board size 152.4 x 25.4 mm -> 80 x 36.4 mm
