File: projects/ro/ro.brd (EAGLE design)
At the start: 80 x 66 mm, 7 parts, among them IC1 MEGA8-P, IC2 MAX6675, Q1 16MHz

Commit message: ds
Parts:
- added C4, C6: 1uF, resistor:C0805
- added C5: 100nF, resistor:C0805
- added D1, D2: 1N4148, adafruit:SMADIODE
- added IC3: 74HCT14N, 74xx-eu:DIL14
- added R1, R2: 82K, resistor:R0805
- added R3, R4: 18K, resistor:R0805
- added S1, S2, S3: (no value), adafruit:B3F-31XX
Connections:
- new net N$3: D1.A, R1.2, R3.1, S1.2
- new net N$4: D2.A, R2.2, R4.1, S2.2
- new net N$5: C4.1, D1.C, IC3.13, R3.2
- new net N$6: C6.1, D2.C, IC3.11, R4.2
- net 2: now also IC3.12
- net 3: now also IC3.10
- net GND: now also C4.2, C5.2, C6.2, IC3.7, S1.1, S2.1, S3.1
- net RESET: now also S3.2
- net VCC: now also C5.1, IC3.14, R1.1, R2.1
Routing:
- net VCC: track 53.9 -> 129.2 mm
- net N$5: track 0.00 -> 60.0 mm
- net N$6: track 0.00 -> 55.5 mm
- net 2: track 0.00 -> 33.3 mm
- net 3: track 0.00 -> 32.0 mm
- net GND: track 84.8 -> 113.7 mm
- net RESET: track 0.00 -> 20.1 mm
- net N$4: track 0.00 -> 18.9 mm
- net N$3: track 0.00 -> 18.5 mm
- added copper zone on layer 1, net GND

Commit message: more design
Parts:
- added U$1: (no value), adafruit:TC33X
- added X1: HD44780LCD-1602, adafruit:LCD1602
- moved S1 68.6 mm to (76.0, 6.00), turned to 90 degrees
- moved R1 65.0 mm to (70.0, 4.00)
- moved R3 57.3 mm to (70.0, 9.00), turned to 180 degrees
- moved D1 55.5 mm to (65.0, 6.00), turned to 90 degrees
- moved S2 52.2 mm to (76.0, 17.0), turned to 90 degrees
- moved R2 46.1 mm to (70.0, 15.0)
- moved C4 44.7 mm to (61.0, 11.0), turned to 90 degrees
- moved C2 41.0 mm to (45.0, 7.00)
- moved D2 39.6 mm to (65.0, 17.0), turned to 90 degrees
- moved R4 38.6 mm to (70.0, 19.0), turned to 180 degrees
- moved IC2 38.3 mm to (16.0, 6.00), turned to 0 degrees
- moved C6 32.0 mm to (61.0, 19.0), turned to 270 degrees
- moved C1 25.6 mm to (25.0, 7.00)
- moved Q1 24.6 mm to (35.0, 7.00), turned to 180 degrees
- moved C5 21.5 mm to (59.0, 4.00)
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Connections:
- new net N$11: U$1.2, X1.3
- net 10: now also X1.12
- net 11: now also X1.13
- net 12: now also X1.14
- net 7: now also X1.4
- net 8: now also X1.6
- net 9: now also X1.11
- net GND: now also U$1.3, X1.1, X1.16, X1.5
- net VCC: now also U$1.1, X1.15, X1.2
Routing:
- net VCC: track 129.2 -> 0.00 mm
- net GND: track 113.7 -> 0.00 mm
- net N$5: track 60.0 -> 0.00 mm
- net N$6: track 55.5 -> 0.00 mm
- net T+: track 39.4 -> 0.00 mm
- net 2: track 33.3 -> 0.00 mm
- net 3: track 32.0 -> 0.00 mm
- net RESET: track 20.1 -> 0.00 mm
- net N$4: track 18.9 -> 0.00 mm
- net A3: track 18.6 -> 0.00 mm
- net N$3: track 18.5 -> 0.00 mm
- net N$2: track 17.4 -> 0.00 mm
- net N$1: track 16.8 -> 0.00 mm
- net A5: track 12.9 -> 0.00 mm
- net A4: track 5.39 -> 0.00 mm
- removed copper zone on layer 1, net GND
Other:
- board size 80 x 66 mm -> 80 x 36 mm
