File: projects/ro/ro.sch (EAGLE design)
At the start: 7 parts, among them IC1 MEGA8-P, IC2 MAX6675, Q1 16MHz

Commit message: ds
Parts:
- added C4, C6: 1uF, resistor:C-USC0805
- added C5: 100nF, resistor:C-USC0805
- added D1, D2: 1N4148, adafruit:DIODESMA
- added IC3: 74HCT14N, 74xx-eu:74HCT14N
- added R1, R2: 82K, resistor:R-US_R0805
- added R3, R4: 18K, resistor:R-US_R0805
- added S1, S2, S3: (no value), adafruit:31-XX
Connections:
- new net N$3: D1.A, R1.2, R3.1, S1.S
- new net N$4: D2.A, R2.2, R4.1, S2.S
- new net N$5: C4.1, D1.C, IC3A.I, R3.2
- new net N$6: C6.1, D2.C, IC3B.I, R4.2
- net 2: now also IC3A.O
- net 3: now also IC3B.O
- net GND: now also C4.2, C5.2, C6.2, IC3P.GND, S1.P, S2.P, S3.P
- net RESET: now also S3.S
- net VCC: now also C5.1, IC3P.VCC, R1.1, R2.1

Commit message: more design
Parts:
- added U$1: (no value), adafruit:TRIMPOTTC33X
- added X1: HD44780LCD-1602, adafruit:HD44780LCD-1602
Connections:
- new net N$11: U$1.S, X1.VO
- net 10: now also X1.DB5
- net 11: now also X1.DB6
- net 12: now also X1.DB7
- net 7: now also X1.RS
- net 8: now also X1.E
- net 9: now also X1.DB4
- net GND: now also U$1.E, X1.K, X1.RW, X1.VSS
- net VCC: now also U$1.A, X1.A, X1.VDD
Changed lines of the file:
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@@
 <part name="S3" library="adafruit" deviceset="31-XX" device=""/>
 <part name="GND10" library="supply1" deviceset="GND" device=""/>
+<part name="X1" library="adafruit" deviceset="HD44780LCD" device="-1602"/>
+<part name="P+7" library="supply1" deviceset="VCC" device=""/>
+<part name="P+8" library="supply1" deviceset="VCC" device=""/>
+<part name="GND11" library="supply1" deviceset="GND" device=""/>
+<part name="GND12" library="supply1" deviceset="GND" device=""/>
+<part name="FRAME4" library="frames" deviceset="A4-SMALL-DOCFIELD" device=""/>
+<part name="GND13" library="supply1" deviceset="GND" device=""/>
+<part name="U$1" library="adafruit" deviceset="TRIMPOT" device="TC33X"/>
+<part name="P+9" library="supply1" deviceset="VCC" device=""/>
+<part name="GND14" library="supply1" deviceset="GND" device=""/>
 </parts>
 <sheets>
@@
 </segment>
 </net>
+</nets>
+</sheet>
+<sheet>
+<plain>
+</plain>
+<instances>
+<instance part="X1" gate="G$1" x="71.12" y="78.74" rot="R180"/>
+<instance part="P+7" gate="VCC" x="55.88" y="50.8" rot="R90"/>
+<instance part="P+8" gate="VCC" x="93.98" y="48.26" rot="R270"/>
+<instance part="GND11" gate="1" x="53.34" y="55.88" rot="R270"/>
+<instance part="GND12" gate="1" x="96.52" y="55.88" rot="R90"/>
+<instance part="FRAME4" gate="/1" x="0" y="0"/>
+<instance part="GND13" gate="1" x="83.82" y="53.34"/>
+<instance part="U$1" gate="G$1" x="88.9" y="40.64" rot="R90"/>
+<instance part="P+9" gate="VCC" x="99.06" y="40.64" rot="R270"/>
+<instance part="GND14" gate="1" x="78.74" y="40.64" rot="R270"/>
+</instances>
+<busses>
+</busses>
+<nets>
+<net name="GND" class="0">
+<segment>
+<pinref part="X1" gate="G$1" pin="VSS"/>
+<pinref part="GND12" gate="1" pin="GND"/>
+<wire x1="93.98" y1="60.96" x2="93.98" y2="55.88" width="0.1524" layer="91"/>
+</segment>
+<segment>
+<pinref part="X1" gate="G$1" pin="K"/>
+<pinref part="GND11" gate="1" pin="GND"/>
+<wire x1="55.88" y1="60.96" x2="55.88" y2="55.88" width="0.1524" layer="91"/>
+</segment>
+<segment>
+<pinref part="X1" gate="G$1" pin="RW"/>
+<wire x1="83.82" y1="60.96" x2="83.82" y2="55.88" width="0.1524" layer="91"/>
+<pinref part="GND13" gate="1" pin="GND"/>
+</segment>
+<segment>
+<pinref part="U$1" gate="G$1" pin="E"/>
+<wire x1="83.82" y1="40.64" x2="81.28" y2="40.64" width="0.1524" layer="91"/>
+<pinref part="GND14" gate="1" pin="GND"/>
+</segment>
+</net>
+<net name="VCC" class="0">
+<segment>
+<pinref part="X1" gate="G$1" pin="A"/>
+<pinref part="P+7" gate="VCC" pin="VCC"/>
+<wire x1="58.42" y1="60.96" x2="58.42" y2="50.8" width="0.1524" layer="91"/>
+</segment>
+<segment>
+<pinref part="X1" gate="G$1" pin="VDD"/>
+<pinref part="P+8" gate="VCC" pin="VCC"/>
+<wire x1="91.44" y1="60.96" x2="91.44" y2="48.26" width="0.1524" layer="91"/>
+</segment>
+<segment>
+<pinref part="U$1" gate="G$1" pin="A"/>
+<wire x1="93.98" y1="40.64" x2="96.52" y2="40.64" width="0.1524" layer="91"/>
+<pinref part="P+9" gate="VCC" pin="VCC"/>
+</segment>
+</net>
+<net name="12" class="0">
+<segment>
+<pinref part="X1" gate="G$1" pin="DB7"/>
+<wire x1="60.96" y1="60.96" x2="60.96" y2="55.88" width="0.1524" layer="91"/>
+<label x="60.96" y="55.88" size="1.778" layer="95" rot="R90"/>
+</segment>
+</net>
+<net name="11" class="0">
+<segment>
+<pinref part="X1" gate="G$1" pin="DB6"/>
+<wire x1="63.5" y1="60.96" x2="63.5" y2="55.88" width="0.1524" layer="91"/>
+<label x="63.5" y="55.88" size="1.778" layer="95" rot="R90"/>
+</segment>
+</net>
+<net name="10" class="0">
+<segment>
+<pinref part="X1" gate="G$1" pin="DB5"/>
+<wire x1="66.04" y1="60.96" x2="66.04" y2="55.88" width="0.1524" layer="91"/>
+<label x="66.04" y="55.88" size="1.778" layer="95" rot="R90"/>
+</segment>
+</net>
+<net name="9" class="0">
+<segment>
+<pinref part="X1" gate="G$1" pin="DB4"/>
+<wire x1="68.58" y1="60.96" x2="68.58" y2="55.88" width="0.1524" layer="91"/>
+<label x="68.58" y="55.88" size="1.778" layer="95" rot="R90"/>
+</segment>
+</net>
+<net name="N$11" class="0">
+<segment>
+<pinref part="X1" gate="G$1" pin="VO"/>
+<pinref part="U$1" gate="G$1" pin="S"/>
+<wire x1="88.9" y1="60.96" x2="88.9" y2="45.72" width="0.1524" layer="91"/>
+</segment>
+</net>
+<net name="7" class="0">
+<segment>
+<pinref part="X1" gate="G$1" pin="RS"/>
+<wire x1="86.36" y1="60.96" x2="86.36" y2="55.88" width="0.1524" layer="91"/>
+<label x="86.36" y="55.88" size="1.778" layer="95" rot="R90"/>
+</segment>
+</net>
+<net name="8" class="0">
+<segment>
+<pinref part="X1" gate="G$1" pin="E"/>
+<wire x1="81.28" y1="60.96" x2="81.28" y2="55.88" width="0.1524" layer="91"/>
+<label x="81.28" y="55.88" size="1.778" layer="95" rot="R90"/>
+</segment>
+</net>
